File: CAN Hat.brd (EAGLE design)
At the start: 56 x 65 mm, 33 parts, among them J1 RASPBERRYPI-40-PIN-GPIO_PTH_N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, Q2 310mA/60V/1.6Ω, Q3 310mA/60V/1.6Ω, U1 MCP2515, U2 MCP2551, X1 C-GRID-03-70543

Commit message: CAN monitor updates
Parts:
- added J8: (no value), SparkFun-Connectors:SCREWTERMINAL-3.5MM-2
- moved R7 0.64 mm to (19.1, 31.1)
Connections:
- net +5V: now also J8.2
- net GND: now also J8.1
Routing:
- net +5V: track 106.9 -> 123.7 mm
- net N$5: track 5.06 -> 4.43 mm
Changed lines of the file:
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@@
 <element name="J4" library="SparkFun-Connectors" package="1X01" value="" x="25.4" y="33.02"/>
 <element name="J5" library="SparkFun-Connectors" package="1X01" value="" x="29.21" y="35.56"/>
-<element name="R7" library="resistor" package="R1206" value="" x="19.05" y="31.75" rot="MR180"/>
+<element name="R7" library="resistor" package="R1206" value="" x="19.05" y="31.115" rot="MR180"/>
 <element name="LED4" library="led" package="LED3MM" value="" x="15.875" y="27.94" smashed="yes">
 <attribute name="VALUE" x="17.78" y="26.289" size="1.27" layer="27" ratio="10"/>
@@
 <attribute name="NAME" x="11.43" y="33.02" size="1.27" layer="25" rot="R270"/>
 <attribute name="VALUE" x="7.62" y="34.29" size="1.27" layer="27" rot="R270"/>
+</element>
+<element name="J8" library="SparkFun-Connectors" package="SCREWTERMINAL-3.5MM-2" value="" x="16.51" y="60.96" rot="R180">
+<attribute name="PROD_ID" value="CONN-08399" x="16.51" y="60.96" size="1.778" layer="27" rot="R180" display="off"/>
 </element>
 </elements>
@@
 <contactref element="J7" pad="1"/>
 <via x="6.35" y="35.56" extent="1-16" drill="0.9"/>
+<contactref element="J8" pad="1"/>
+<via x="8.89" y="60.96" extent="1-16" drill="0.9"/>
 </signal>
 <signal name="+5V">
@@
 <contactref element="J1" pad="4"/>
 <contactref element="X1" pad="1"/>
-<wire x1="54.61" y1="57.15" x2="54.61" y2="54.61" width="0.4064" layer="16"/>
 <wire x1="21.85" y1="34.925" x2="20.955" y2="34.925" width="0.4064" layer="16"/>
 <wire x1="20.955" y1="34.925" x2="20.32" y2="35.56" width="0.4064" layer="16"/>
@@
 <wire x1="22.355" y1="40.005" x2="22.355" y2="43.685" width="0.4064" layer="16"/>
 <wire x1="22.355" y1="43.685" x2="21.59" y2="44.45" width="0.4064" layer="16"/>
-<wire x1="54.61" y1="57.15" x2="54.61" y2="57.785" width="0.4064" layer="16"/>
-<wire x1="54.61" y1="57.785" x2="53.34" y2="59.055" width="0.4064" layer="16"/>
-<wire x1="53.34" y1="59.055" x2="41.91" y2="59.055" width="0.4064" layer="16"/>
-<wire x1="41.91" y1="59.055" x2="28.575" y2="59.055" width="0.4064" layer="16"/>
-<wire x1="28.575" y1="59.055" x2="21.59" y2="52.07" width="0.4064" layer="16"/>
 <wire x1="21.59" y1="52.07" x2="21.59" y2="44.45" width="0.4064" layer="16"/>
 <contactref element="R7" pad="2"/>
-<wire x1="20.472" y1="31.75" x2="20.472" y2="34.442" width="0.4064" layer="16"/>
+<wire x1="20.472" y1="31.115" x2="20.472" y2="34.442" width="0.4064" layer="16"/>
 <wire x1="20.472" y1="34.442" x2="20.955" y2="34.925" width="0.4064" layer="16"/>
 <contactref element="C4" pad="2"/>
@@
 <wire x1="40.64" y1="40.64" x2="41.78" y2="40.64" width="0.4064" layer="16"/>
 <wire x1="41.78" y1="40.64" x2="41.91" y2="40.77" width="0.4064" layer="16"/>
+<contactref element="J8" pad="2"/>
+<wire x1="13.01" y1="60.96" x2="13.01" y2="60.65" width="0.8128" layer="16"/>
+<wire x1="13.01" y1="60.65" x2="15.24" y2="58.42" width="0.8128" layer="16"/>
+<wire x1="15.24" y1="58.42" x2="27.94" y2="58.42" width="0.8128" layer="16"/>
+<wire x1="27.94" y1="58.42" x2="28.575" y2="59.055" width="0.8128" layer="16"/>
+<wire x1="54.61" y1="54.61" x2="54.61" y2="57.15" width="0.8128" layer="16"/>
+<wire x1="54.61" y1="57.15" x2="54.61" y2="57.785" width="0.8128" layer="16"/>
+<wire x1="54.61" y1="57.785" x2="53.34" y2="59.055" width="0.8128" layer="16"/>
+<wire x1="53.34" y1="59.055" x2="41.91" y2="59.055" width="0.8128" layer="16"/>
+<wire x1="41.91" y1="59.055" x2="28.575" y2="59.055" width="0.8128" layer="16"/>
+<wire x1="21.59" y1="52.07" x2="27.94" y2="58.42" width="0.4064" layer="16"/>
 </signal>
 <signal name="N$3">
@@
 <contactref element="R7" pad="1"/>
 <contactref element="LED4" pad="A"/>
-<wire x1="14.605" y1="27.94" x2="14.605" y2="28.727" width="0.4064" layer="16"/>
-<wire x1="14.605" y1="28.727" x2="17.628" y2="31.75" width="0.4064" layer="16"/>
+<wire x1="17.628" y1="31.115" x2="17.628" y2="30.963" width="0.4064" layer="16"/>
+<wire x1="17.628" y1="30.963" x2="14.605" y2="27.94" width="0.4064" layer="16"/>
 </signal>
 <signal name="N$26">
