File: CAN Hat.sch (EAGLE design)
At the start: 33 parts, among them J1 RASPBERRYPI-40-PIN-GPIO_PTH_N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, Q2 310mA/60V/1.6Ω, Q3 310mA/60V/1.6Ω, U1 MCP2515, U2 MCP2551, X1 C-GRID-03-70543

Commit message: CAN monitor updates
Parts:
- added J8: (no value), SparkFun-Connectors:CONN_023.5MM
Connections:
- net +5V: now also J8.2
- net GND: now also J8.1
Changed lines of the file:
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@@
 <part name="C5" library="resistor" deviceset="C-EU" device="C1206"/>
 <part name="R10" library="resistor" deviceset="R-US_" device="R1206"/>
+<part name="J8" library="SparkFun-Connectors" deviceset="CONN_02" device="3.5MM"/>
+<part name="SUPPLY24" library="supply2" deviceset="+5V" device=""/>
+<part name="SUPPLY25" library="supply2" deviceset="GND" device=""/>
 </parts>
 <sheets>
@@
 <instance part="C5" gate="G$1" x="154.94" y="50.8" rot="R180"/>
 <instance part="R10" gate="G$1" x="154.94" y="43.18" rot="R270"/>
+<instance part="J8" gate="G$1" x="55.88" y="81.28"/>
+<instance part="SUPPLY24" gate="+5V" x="63.5" y="86.36"/>
+<instance part="SUPPLY25" gate="GND" x="63.5" y="78.74"/>
 </instances>
 <busses>
@@
 <pinref part="SUPPLY23" gate="GND" pin="GND"/>
 </segment>
+<segment>
+<pinref part="J8" gate="G$1" pin="1"/>
+<pinref part="SUPPLY25" gate="GND" pin="GND"/>
+</segment>
 </net>
 <net name="+5V" class="0">
@@
 <pinref part="SUPPLY22" gate="+5V" pin="+5V"/>
 </segment>
+<segment>
+<pinref part="J8" gate="G$1" pin="2"/>
+<pinref part="SUPPLY24" gate="+5V" pin="+5V"/>
+</segment>
 </net>
